File: kicad/le_chiff_ble/_autosave-le_chiff_ble.kicad_pcb (KiCad board)
At the start: 2 copper layers, 228.4 x 85 mm, 117 parts, among them J2 BL_CONN, Q1 AO3401A, SW1 ON_OFF, SW2 SW_RESET, SW3 Rotary_Encoder_Switch, U1 TP4056, U2 MS88SF2, U3 XC6206PxxxMR-Regulator_Linear, U4 DW01A, U5 FS8205, U6 USBLC6-2SC6

Commit message: finished the schematics and the PCB, maybe some silkscreen to come..
Routing:
- net col2: track 242.6 -> 240.5 mm
- net GND: vias 33 -> 31
Other:
- board text added: "die Zivilisation nur eine sehr dünne Decke ist, die sehr schnell abblättert.“ - Fritz Bauer"
- board text added: "„Ich glaube, es ist eine traurige Wahrheit, dass wir unserem Affenzustand noch sehr nahe sind und dass"
Changed lines of the file:
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@@
   (general
     (thickness 1.6)
-    (drawings 78)
-    (tracks 1212)
+    (drawings 80)
+    (tracks 1216)
     (zones 0)
     (modules 117)
@@
   (module graphics:mangoiv (layer B.Cu)
     (at 151.379425 123.443326 270)
-    (fp_text reference G*** (at 0 0 270) (layer B.SilkS) hide
+    (fp_text reference G*** (at 0 0 270) (layer B.Mask) hide
       (effects (font (size 1.524 1.524) (thickness 0.3)) (justify mirror))
     )
-    (fp_text value LOGO (at 0.75 0 270) (layer B.SilkS) hide
+    (fp_text value LOGO (at 0.75 0 270) (layer B.Mask) hide
       (effects (font (size 1.524 1.524) (thickness 0.3)) (justify mirror))
     )
@@
     )
   )
+  (gr_text "die Zivilisation nur eine sehr dünne Decke ist, \ndie sehr schnell abblättert.“  -  Fritz Bauer" (at 114.379425 62.443326 -11) (layer B.Mask)
+    (effects (font (size 1 1) (thickness 0.2)) (justify mirror))
+  )
+  (gr_text "„Ich glaube, es ist eine traurige Wahrheit, dass wir \nunserem Affenzustand noch sehr nahe sind und dass " (at 177.129425 62.443326 11) (layer B.Mask)
+    (effects (font (size 1 1) (thickness 0.2)) (justify mirror))
+  )
   (gr_text RESET (at 147.474663 91.943326) (layer B.SilkS)
     (effects (font (size 1 1) (thickness 0.25)) (justify left mirror))
@@
   (segment (start 157.739425 118.553326) (end 158.379425 119.193326) (width 0.381) (layer F.Cu) (net 3))
   (segment (start 158.379425 119.193326) (end 160.379425 119.193326) (width 0.381) (layer F.Cu) (net 3))
-  (via (at 132.879425 67.943326) (size 0.8) (drill 0.4) (layers F.Cu B.Cu) (net 3))
   (via (at 94.879425 58.693326) (size 0.8) (drill 0.4) (layers F.Cu B.Cu) (net 3))
   (via (at 128.629425 107.193326) (size 0.8) (drill 0.4) (layers F.Cu B.Cu) (net 3))
@@
   (via (at 137.879425 74.943326) (size 0.8) (drill 0.4) (layers F.Cu B.Cu) (net 3))
   (via (at 119.579425 136.873666) (size 0.8) (drill 0.4) (layers F.Cu B.Cu) (net 3))
-  (via (at 113.379425 67.693326) (size 0.8) (drill 0.4) (layers F.Cu B.Cu) (net 3))
-  (via (at 94.629425 66.193326) (size 0.8) (drill 0.4) (layers F.Cu B.Cu) (net 3))
   (via (at 130.129425 74.443326) (size 0.8) (drill 0.4) (layers F.Cu B.Cu) (net 3))
+  (via (at 112.129425 75.693326) (size 0.8) (drill 0.4) (layers F.Cu B.Cu) (net 3))
   (segment (start 142.879425 66.693326) (end 141.879425 67.693326) (width 0.381) (layer F.Cu) (net 4))
   (segment (start 145.690425 66.693326) (end 142.879425 66.693326) (width 0.381) (layer F.Cu) (net 4))
@@
   (segment (start 230.379425 73.593326) (end 237.379425 80.593326) (width 0.25) (layer B.Cu) (net 14))
   (segment (start 217.379425 73.593326) (end 230.379425 73.593326) (width 0.25) (layer B.Cu) (net 14))
-  (segment (start 126.379425 82.843326) (end 110.129425 82.843326) (width 0.25) (layer B.Cu) (net 14))
-  (segment (start 128.879425 85.343326) (end 126.379425 82.843326) (width 0.25) (layer B.Cu) (net 14))
-  (segment (start 102.279425 75.843326) (end 91.879425 75.843326) (width 0.25) (layer B.Cu) (net 14))
-  (segment (start 109.279425 82.843326) (end 102.279425 75.843326) (width 0.25) (layer B.Cu) (net 14))
-  (segment (start 110.129425 82.843326) (end 109.279425 82.843326) (width 0.25) (layer B.Cu) (net 14))
   (segment (start 75.379219 75.343532) (end 72.379425 78.343326) (width 0.25) (layer B.Cu) (net 14))
   (segment (start 91.379631 75.343532) (end 75.379219 75.343532) (width 0.25) (layer B.Cu) (net 14))
@@
   (via (at 162.979425 85.343326) (size 0.8) (drill 0.4) (layers F.Cu B.Cu) (net 14))
   (segment (start 161.379425 85.343326) (end 162.979425 85.343326) (width 0.25) (layer B.Cu) (net 14))
-  (segment (start 159.354426 83.318327) (end 161.379425 85.343326) (width 0.25) (layer B.Cu) (net 14))
-  (segment (start 130.904424 83.318327) (end 159.354426 83.318327) (width 0.25) (layer B.Cu) (net 14))
-  (segment (start 128.879425 85.343326) (end 130.904424 83.318327) (width 0.25) (layer B.Cu) (net 14))
   (segment (start 157.019425 124.053326) (end 160.204413 120.868338) (width 0.25) (layer F.Cu) (net 14))
   (segment (start 153.629425 124.053326) (end 157.019425 124.053326) (width 0.25) (layer F.Cu) (net 14))
@@
   (segment (start 167.479425 85.343326) (end 169.979425 82.843326) (width 0.25) (layer B.Cu) (net 14))
   (segment (start 162.979425 85.343326) (end 167.479425 85.343326) (width 0.25) (layer B.Cu) (net 14))
+  (segment (start 121.779425 82.843326) (end 110.129425 82.843326) (width 0.25) (layer B.Cu) (net 14))
+  (segment (start 124.279425 85.343326) (end 121.779425 82.843326) (width 0.25) (layer B.Cu) (net 14))
+  (segment (start 128.879425 85.343326) (end 124.279425 85.343326) (width 0.25) (layer B.Cu) (net 14))
+  (segment (start 99.529425 75.843326) (end 91.879425 75.843326) (width 0.25) (layer B.Cu) (net 14))
+  (segment (start 106.529425 82.843326) (end 99.529425 75.843326) (width 0.25) (layer B.Cu) (net 14))
+  (segment (start 110.129425 82.843326) (end 106.529425 82.843326) (width 0.25) (layer B.Cu) (net 14))
+  (segment (start 128.879425 85.343326) (end 130.115835 85.343326) (width 0.25) (layer B.Cu) (net 14))
+  (segment (start 130.115835 85.343326) (end 132.140834 83.318327) (width 0.25) (layer B.Cu) (net 14))
+  (segment (start 132.140834 83.318327) (end 159.354426 83.318327) (width 0.25) (layer B.Cu) (net 14))
+  (segment (start 159.354426 83.318327) (end 161.379425 85.343326) (width 0.25) (layer B.Cu) (net 14))
   (segment (start 41.416788 83.055514) (end 40.285035 83.055514) (width 0.25) (layer B.Cu) (net 15))
   (segment (start 42.997952 81.47435) (end 41.416788 83.055514) (width 0.25) (layer B.Cu) (net 15))
@@
   (segment (start 118.661044 69.998903) (end 117.340595 69.998903) (width 0.25) (layer B.Cu) (net 30))
   (segment (start 121.531677 67.12827) (end 118.661044 69.998903) (width 0.25) (layer B.Cu) (net 30))
-  (segment (start 126.439708 82.043326) (end 128.879425 82.043326) (width 0.25) (layer B.Cu) (net 30))
-  (segment (start 117.340595 72.944213) (end 126.439708 82.043326) (width 0.25) (layer B.Cu) (net 30))
-  (segment (start 117.340595 69.998903) (end 117.340595 72.944213) (width 0.25) (layer B.Cu) (net 30))
+  (segment (start 128.829414 81.993315) (end 128.879425 82.043326) (width 0.25) (layer B.Cu) (net 30))
+  (segment (start 117.420526 73.024144) (end 126.389697 81.993315) (width 0.25) (layer B.Cu) (net 30))
+  (segment (start 117.420526 70.078834) (end 117.420526 73.024144) (width 0.25) (layer B.Cu) (net 30))
+  (segment (start 126.389697 81.993315) (end 128.829414 81.993315) (width 0.25) (layer B.Cu) (net 30))
+  (segment (start 117.340595 69.998903) (end 117.420526 70.078834) (width 0.25) (layer B.Cu) (net 30))
   (segment (start 117.628903 87.617436) (end 116.49715 87.617436) (width 0.25) (layer B.Cu) (net 31))
   (segment (start 119.210067 86.036272) (end 117.628903 87.617436) (width 0.25) (layer B.Cu) (net 31))
@@
   (segment (start 145.625427 74.393326) (end 139.825427 80.193326) (width 0.25) (layer F.Cu) (net 57))
   (segment (start 150.129425 74.393326) (end 145.625427 74.393326) (width 0.25) (layer F.Cu) (net 57))
-  (segment (start 107.879425 63.193326) (end 91.741677 63.193326) (width 0.25) (layer B.Cu) (net 57))
-  (segment (start 110.379425 65.693326) (end 107.879425 63.193326) (width 0.25) (layer B.Cu) (net 57))
-  (segment (start 126.129425 65.693326) (end 110.379425 65.693326) (width 0.25) (layer B.Cu) (net 57))
-  (segment (start 134.129425 73.693326) (end 126.129425 65.693326) (width 0.25) (layer B.Cu) (net 57))
+  (segment (start 110.379425 68.193326) (end 105.379425 63.193326) (width 0.25) (layer B.Cu) (net 57))
+  (segment (start 130.379425 84.443326) (end 124.379425 84.443326) (width 0.25) (layer B.Cu) (net 57))
+  (segment (start 132.379425 82.443326) (end 130.379425 84.443326) (width 0.25) (layer B.Cu) (net 57))
+  (segment (start 110.379425 70.443326) (end 110.379425 68.193326) (width 0.25) (layer B.Cu) (net 57))
+  (segment (start 124.379425 84.443326) (end 110.379425 70.443326) (width 0.25) (layer B.Cu) (net 57))
+  (segment (start 134.129425 82.443326) (end 132.379425 82.443326) (width 0.25) (layer B.Cu) (net 57))
   (segment (start 91.741677 63.193326) (end 89.002572 60.454221) (width 0.25) (layer B.Cu) (net 57))
-  (segment (start 134.129425 82.443326) (end 134.129425 73.693326) (width 0.25) (layer B.Cu) (net 57))
+  (segment (start 105.379425 63.193326) (end 91.741677 63.193326) (width 0.25) (layer B.Cu) (net 57))
   (segment (start 135.039425 121.853326) (end 131.063393 117.877294) (width 0.25) (layer F.Cu) (net 58))
   (via (at 131.063393 117.877294) (size 0.8) (drill 0.4) (layers F.Cu B.Cu) (net 58))
