File: kicad/le_chiff_ble/le_chiff_ble.sch (KiCad schematic (older format))
At the start: 114 parts, among them J2 BL_CONN, Q1 AO3401A, SW1 ON_OFF, SW2 SW_RESET, SW3 Rotary_Encoder_Switch, U1 TP4056, U2 MS88SF2, U3 XC6206PxxxMR-Regulator_Linear, U4 DW01A, U5 FS8205, U6 USBLC6-2SC6

Commit message: changed paths to be relative
Parts:
- MX1, MX10, MX11, MX12, MX13, MX14, MX15, MX16, MX17, MX18, MX19, MX2, MX20, MX21, MX22, MX23, MX24, MX25, MX26, MX27, MX28, MX29, MX3, MX30, MX31, MX32, MX33, MX34, MX35, MX4, MX5, MX6, MX7, MX8, MX9: symbol kicad-keyboard-parts:MX_LED -> le_chiff_ble-rescue:MX_LED-kicad-keyboard-parts
- OL1: symbol kbd:OLED -> le_chiff_ble-rescue:OLED-kbd
- U1: symbol tp4056:TP4056 -> le_chiff_ble-rescue:TP4056-tp4056
- U2: symbol MINEW_MS88SF2:MS88SF2 -> le_chiff_ble-rescue:MS88SF2-MINEW_MS88SF2
- U3: symbol kicad-keyboard-parts:XC6206PxxxMR-Regulator_Linear -> le_chiff_ble-rescue:XC6206PxxxMR-Regulator_Linear-kicad-keyboard-parts
- U4: symbol kicad-keyboard-parts:DW01A -> le_chiff_ble-rescue:DW01A-kicad-keyboard-parts
- U5: symbol kicad-keyboard-parts:FS8205 -> le_chiff_ble-rescue:FS8205-kicad-keyboard-parts
- USB1: symbol keebio:HRO-TYPE-C-31-M-12 -> le_chiff_ble-rescue:HRO-TYPE-C-31-M-12-keebio
Changed lines of the file:
@@
 $EndDescr
 $Comp
-L MINEW_MS88SF2:MS88SF2 U2
+L le_chiff_ble-rescue:MS88SF2-MINEW_MS88SF2 U2
 U 1 1 60C5FFDB
 P 2450 2150
@@
 	10200 1100 10600 1100
 $Comp
-L kicad-keyboard-parts:DW01A U4
+L le_chiff_ble-rescue:DW01A-kicad-keyboard-parts U4
 U 1 1 60D64A0D
 P 3700 5300
@@
 $EndComp
 $Comp
-L kicad-keyboard-parts:FS8205 U5
+L le_chiff_ble-rescue:FS8205-kicad-keyboard-parts U5
 U 1 1 60D6A758
 P 3700 5950
@@
 	4300 5350 4400 5350
 $Comp
-L kicad-keyboard-parts:XC6206PxxxMR-Regulator_Linear U3
+L le_chiff_ble-rescue:XC6206PxxxMR-Regulator_Linear-kicad-keyboard-parts U3
 U 1 1 60D92CBC
 P 3200 7250
@@
 connector to flash the bootloader
 $Comp
-L kbd:OLED OL1
+L le_chiff_ble-rescue:OLED-kbd OL1
 U 1 1 60ECBCE6
 P 10350 2100
@@
 col0
 $Comp
-L kicad-keyboard-parts:MX_LED MX1
+L le_chiff_ble-rescue:MX_LED-kicad-keyboard-parts MX1
 U 1 1 60F59542
 P 5400 3950
@@
 $EndComp
 $Comp
-L kicad-keyboard-parts:MX_LED MX2
+L le_chiff_ble-rescue:MX_LED-kicad-keyboard-parts MX2
 U 1 1 60F636D1
 P 5400 4650
@@
 $EndComp
 $Comp
-L kicad-keyboard-parts:MX_LED MX3
+L le_chiff_ble-rescue:MX_LED-kicad-keyboard-parts MX3
 U 1 1 60F69877
 P 5400 5300
@@
 $EndComp
 $Comp
-L kicad-keyboard-parts:MX_LED MX4
+L le_chiff_ble-rescue:MX_LED-kicad-keyboard-parts MX4
 U 1 1 60F6FD2C
 P 5850 3950
@@
 $EndComp
 $Comp
-L kicad-keyboard-parts:MX_LED MX5
+L le_chiff_ble-rescue:MX_LED-kicad-keyboard-parts MX5
 U 1 1 60F6FD38
 P 5850 4650
@@
 $EndComp
 $Comp
-L kicad-keyboard-parts:MX_LED MX6
+L le_chiff_ble-rescue:MX_LED-kicad-keyboard-parts MX6
 U 1 1 60F6FD44
 P 5850 5300
@@
 $EndComp
 $Comp
-L kicad-keyboard-parts:MX_LED MX7
+L le_chiff_ble-rescue:MX_LED-kicad-keyboard-parts MX7
 U 1 1 60F78131
 P 6300 3950
@@
 $EndComp
 $Comp
-L kicad-keyboard-parts:MX_LED MX8
+L le_chiff_ble-rescue:MX_LED-kicad-keyboard-parts MX8
 U 1 1 60F7813D
 P 6300 4650
@@
 $EndComp
 $Comp
-L kicad-keyboard-parts:MX_LED MX9
+L le_chiff_ble-rescue:MX_LED-kicad-keyboard-parts MX9
 U 1 1 60F78149
 P 6300 5300
@@
 $EndComp
 $Comp
-L kicad-keyboard-parts:MX_LED MX10
+L le_chiff_ble-rescue:MX_LED-kicad-keyboard-parts MX10
 U 1 1 60F78155
 P 6750 3950
@@
 $EndComp
 $Comp
-L kicad-keyboard-parts:MX_LED MX11
+L le_chiff_ble-rescue:MX_LED-kicad-keyboard-parts MX11
 U 1 1 60F78161
 P 6750 4650
@@
 $EndComp
 $Comp
-L kicad-keyboard-parts:MX_LED MX12
+L le_chiff_ble-rescue:MX_LED-kicad-keyboard-parts MX12
 U 1 1 60F7816D
 P 6750 5300
@@
 $EndComp
 $Comp
-L kicad-keyboard-parts:MX_LED MX14
+L le_chiff_ble-rescue:MX_LED-kicad-keyboard-parts MX14
 U 1 1 60F862AC
 P 7200 3950
@@
 $EndComp
 $Comp
-L kicad-keyboard-parts:MX_LED MX15
+L le_chiff_ble-rescue:MX_LED-kicad-keyboard-parts MX15
 U 1 1 60F862B8
 P 7200 4650
@@
 $EndComp
 $Comp
-L kicad-keyboard-parts:MX_LED MX16
+L le_chiff_ble-rescue:MX_LED-kicad-keyboard-parts MX16
 U 1 1 60F862C4
 P 7200 5300
@@
 $EndComp
 $Comp
-L kicad-keyboard-parts:MX_LED MX18
+L le_chiff_ble-rescue:MX_LED-kicad-keyboard-parts MX18
 U 1 1 60F862D0
 P 7650 3950
@@
 $EndComp
 $Comp
-L kicad-keyboard-parts:MX_LED MX19
+L le_chiff_ble-rescue:MX_LED-kicad-keyboard-parts MX19
 U 1 1 60F862DC
 P 7650 4650
@@
 $EndComp
 $Comp
-L kicad-keyboard-parts:MX_LED MX20
+L le_chiff_ble-rescue:MX_LED-kicad-keyboard-parts MX20
 U 1 1 60F862E8
 P 7650 5300
@@
 $EndComp
 $Comp
-L kicad-keyboard-parts:MX_LED MX22
+L le_chiff_ble-rescue:MX_LED-kicad-keyboard-parts MX22
 U 1 1 60F862F4
 P 8100 3950
@@
 $EndComp
 $Comp
-L kicad-keyboard-parts:MX_LED MX23
+L le_chiff_ble-rescue:MX_LED-kicad-keyboard-parts MX23
 U 1 1 60F86300
 P 8100 4650
@@
 $EndComp
 $Comp
-L kicad-keyboard-parts:MX_LED MX24
+L le_chiff_ble-rescue:MX_LED-kicad-keyboard-parts MX24
 U 1 1 60F8630C
 P 8100 5300
@@
 $EndComp
 $Comp
-L kicad-keyboard-parts:MX_LED MX26
+L le_chiff_ble-rescue:MX_LED-kicad-keyboard-parts MX26
 U 1 1 60F86318
 P 8550 3950
@@
 $EndComp
 $Comp
-L kicad-keyboard-parts:MX_LED MX27
+L le_chiff_ble-rescue:MX_LED-kicad-keyboard-parts MX27
 U 1 1 60F86324
 P 8550 4650
@@
 $EndComp
 $Comp
-L kicad-keyboard-parts:MX_LED MX28
+L le_chiff_ble-rescue:MX_LED-kicad-keyboard-parts MX28
 U 1 1 60F86330
 P 8550 5300
@@
 $EndComp
 $Comp
-L kicad-keyboard-parts:MX_LED MX29
+L le_chiff_ble-rescue:MX_LED-kicad-keyboard-parts MX29
 U 1 1 60F94005
 P 9000 3950
@@
 $EndComp
 $Comp
-L kicad-keyboard-parts:MX_LED MX30
+L le_chiff_ble-rescue:MX_LED-kicad-keyboard-parts MX30
 U 1 1 60F94011
 P 9000 4650
@@
 $EndComp
 $Comp
-L kicad-keyboard-parts:MX_LED MX31
+L le_chiff_ble-rescue:MX_LED-kicad-keyboard-parts MX31
 U 1 1 60F9401D
 P 9000 5300
@@
 $EndComp
 $Comp
-L kicad-keyboard-parts:MX_LED MX32
+L le_chiff_ble-rescue:MX_LED-kicad-keyboard-parts MX32
 U 1 1 60F94029
 P 9450 3950
@@
 $EndComp
 $Comp
-L kicad-keyboard-parts:MX_LED MX33
+L le_chiff_ble-rescue:MX_LED-kicad-keyboard-parts MX33
 U 1 1 60F94035
 P 9450 4650
@@
 $EndComp
 $Comp
-L kicad-keyboard-parts:MX_LED MX34
+L le_chiff_ble-rescue:MX_LED-kicad-keyboard-parts MX34
 U 1 1 60F94041
 P 9450 5300
@@
 $EndComp
 $Comp
-L kicad-keyboard-parts:MX_LED MX13
+L le_chiff_ble-rescue:MX_LED-kicad-keyboard-parts MX13
 U 1 1 60FAC210
 P 6750 5950
@@
 $EndComp
 $Comp
-L kicad-keyboard-parts:MX_LED MX17
+L le_chiff_ble-rescue:MX_LED-kicad-keyboard-parts MX17
 U 1 1 60FAC21C
 P 7200 5950
@@
 $EndComp
 $Comp
-L kicad-keyboard-parts:MX_LED MX21
+L le_chiff_ble-rescue:MX_LED-kicad-keyboard-parts MX21
 U 1 1 60FAC228
 P 7650 5950
@@
 $EndComp
 $Comp
-L kicad-keyboard-parts:MX_LED MX25
+L le_chiff_ble-rescue:MX_LED-kicad-keyboard-parts MX25
 U 1 1 60FAC234
 P 8100 5950
@@
 $EndComp
 $Comp
-L kicad-keyboard-parts:MX_LED MX35
+L le_chiff_ble-rescue:MX_LED-kicad-keyboard-parts MX35
 U 1 1 60FC6BAD
 P 10700 2850
@@
 swclk
 $Comp
-L tp4056:TP4056 U1
+L le_chiff_ble-rescue:TP4056-tp4056 U1
 U 1 1 6147D430
 P 1850 6300
@@
 	1300 6450 1350 6450
 $Comp
-L keebio:HRO-TYPE-C-31-M-12 USB1
+L le_chiff_ble-rescue:HRO-TYPE-C-31-M-12-keebio USB1
 U 1 1 616F21A5
 P 8150 1800
@@
 	750  6350 750  6400
 $Comp
-L kicad-keyboard-parts:MX_LED MX21
+L le_chiff_ble-rescue:MX_LED-kicad-keyboard-parts MX21
 U 2 1 61D07AA6
 P 850 6250
@@
 	1050 6400 1050 6450
 $Comp
-L kicad-keyboard-parts:MX_LED MX17
+L le_chiff_ble-rescue:MX_LED-kicad-keyboard-parts MX17
 U 2 1 61D1A873
 P 550 6250
