File: kicad/le_chiff_ble/le_chiff_ble.sch (KiCad schematic (older format))
At the start: 114 parts, among them J2 BL_CONN, Q1 AO3401A, SW1 ON_OFF, SW2 SW_RESET, SW3 Rotary_Encoder_Switch, U1 TP4056, U2 MS88SF2, U3 XC6206PxxxMR-Regulator_Linear, U4 DW01A, U5 FS8205, U6 USBLC6-2SC6

Commit message: started rerouting
Connections:
- net col0: now also U2.28 (P0.10); no longer U2.12 (P0.12)
- net col1: now also U2.27 (P0.09); no longer U2.11 (P1.09)
- net col2: now also MX13.1 (COL), U2.24 (P1.00); no longer MX35.1 (COL), SW3.S1, U2.10 (P0.08)
- net col3: now also MX17.1 (COL), U2.21 (P0.20); no longer MX13.1 (COL), U2.19 (P0.15)
- net col4: now also U2.19 (P0.15); no longer MX17.1 (COL), U2.18 (P0.13)
- net col5: now also MX35.1 (COL), SW3.S1, U2.11 (P1.09); no longer MX21.1 (COL), U2.7 (P0.26)
- net col6: now also MX21.1 (COL), U2.10 (P0.08); no longer MX25.1 (COL), U2.5 (P0.29)
- net col7: now also MX25.1 (COL), U2.9 (P0.06); no longer U2.4 (P0.02)
- net col8: now also U2.8 (P0.04); no longer U2.3 (P1.15)
- net col9: now also U2.7 (P0.26); no longer U2.2 (P1.13)
- net encA: now also U2.12 (P0.12); no longer U2.28 (P0.10)
- net encB: now also U2.18 (P0.13); no longer U2.27 (P0.09)
- net row0: now also U2.5 (P0.29); no longer U2.8 (P0.04)
- net row1: now also U2.4 (P0.02); no longer U2.9 (P0.06)
- net row2: now also U2.3 (P1.15); no longer U2.21 (P0.20)
- net row3: now also U2.2 (P1.13); no longer U2.24 (P1.00)
- net at MX28.2 (ROW): no longer D31.2 (A)
Other:
- moved on the sheet: D16, D20, D24, D28, MX13A, MX17A, MX21A, MX25A, MX28A
Changed lines of the file:
@@
 $EndDescr
-$Comp
-L MINEW_MS88SF2:MS88SF2 U2
-U 1 1 60C5FFDB
-P 2450 2150
-F 0 "U2" H 2425 3067 50  0000 C CNN
-F 1 "MS88SF2" H 2425 2976 50  0000 C CNN
-F 2 "ms88sf2_oreore:MINEW_MS88SF2" H 2450 2200 50  0001 C CNN
-F 3 "" H 2450 2200 50  0001 C CNN
-	1    2450 2150
-	1    0    0    -1
-$EndComp
 $Comp
 L Device:R_Small R15
@@
 Text GLabel 4950 1700 0    50   Input ~ 0
 vbus
-$Comp
-L power:GND #PWR0105
-U 1 1 60C8E0D5
-P 1500 1500
-F 0 "#PWR0105" H 1500 1250 50  0001 C CNN
-F 1 "GND" H 1505 1327 50  0000 C CNN
-F 2 "" H 1500 1500 50  0001 C CNN
-F 3 "" H 1500 1500 50  0001 C CNN
-	1    1500 1500
-	1    0    0    -1
-$EndComp
-Wire Wire Line
-	1500 1500 1800 1500
 Text GLabel 3050 2600 2    50   Input ~ 0
 d+
@@
 	0    -1   -1   0
 $EndComp
-$Comp
-L power:GND #PWR0110
-U 1 1 60CBF5F2
-P 1500 2700
-F 0 "#PWR0110" H 1500 2450 50  0001 C CNN
-F 1 "GND" V 1505 2572 50  0000 R CNN
-F 2 "" H 1500 2700 50  0001 C CNN
-F 3 "" H 1500 2700 50  0001 C CNN
-	1    1500 2700
-	0    1    1    0
-$EndComp
-Wire Wire Line
-	1500 2700 1800 2700
 Wire Wire Line
 	1500 2800 1650 2800
@@
 $EndComp
 Connection ~ 1650 2800
-Wire Wire Line
-	1650 2800 1800 2800
 $Comp
 L power:GND #PWR0111
@@
 	1    0    0    -1
 $EndComp
-Wire Wire Line
-	3050 2800 3200 2800
 Connection ~ 3200 2800
 Wire Wire Line
@@
 	1    0    0    -1
 $EndComp
-Text GLabel 3050 1500 2    50   Input ~ 0
+Text GLabel 1800 2600 0    50   Input ~ 0
 encA
-Text GLabel 3050 1600 2    50   Input ~ 0
+Text GLabel 3050 2500 2    50   Input ~ 0
 encB
 Text GLabel 9600 3050 0    50   Input ~ 0
@@
 F 3 "" H 8600 5400 50  0001 C CNN
 	1    8550 5300
-	1    0    0    -1
+	1    0    0    1
 $EndComp
 $Comp
@@
 L kicad-keyboard-parts:MX_LED MX13
 U 1 1 60FAC210
+P 6300 5950
+F 0 "MX13" H 6333 6117 50  0000 C CNN
+F 1 "MX_LED" H 6333 6050 20  0000 C CNN
+F 2 "Keebio-Parts:MX-Alps-Choc-1U-NoLED" H 6350 6050 50  0001 C CNN
+F 3 "" H 6350 6050 50  0001 C CNN
+	1    6300 5950
+	1    0    0    -1
+$EndComp
+$Comp
+L Device:D_Small D16
+U 1 1 60FAC216
+P 6250 6250
+F 0 "D16" V 6296 6180 50  0000 R CNN
+F 1 "D_Small" V 6205 6180 50  0000 R CNN
+F 2 "Diode_SMD:D_SOD-123" V 6250 6250 50  0001 C CNN
+F 3 "~" V 6250 6250 50  0001 C CNN
+	1    6250 6250
+	0    -1   -1   0
+$EndComp
+$Comp
+L kicad-keyboard-parts:MX_LED MX17
+U 1 1 60FAC21C
 P 6750 5950
-F 0 "MX13" H 6783 6117 50  0000 C CNN
+F 0 "MX17" H 6783 6117 50  0000 C CNN
 F 1 "MX_LED" H 6783 6050 20  0000 C CNN
-F 2 "Keebio-Parts:MX-Alps-Choc-1U-NoLED" H 6800 6050 50  0001 C CNN
+F 2 "Keebio-Parts:MX-Alps-Choc-2U-StabFlip" H 6800 6050 50  0001 C CNN
 F 3 "" H 6800 6050 50  0001 C CNN
 	1    6750 5950
@@
 $EndComp
 $Comp
-L Device:D_Small D16
-U 1 1 60FAC216
+L Device:D_Small D20
+U 1 1 60FAC222
 P 6700 6250
-F 0 "D16" V 6746 6180 50  0000 R CNN
+F 0 "D20" V 6746 6180 50  0000 R CNN
 F 1 "D_Small" V 6655 6180 50  0000 R CNN
 F 2 "Diode_SMD:D_SOD-123" V 6700 6250 50  0001 C CNN
@@
 $EndComp
 $Comp
-L kicad-keyboard-parts:MX_LED MX17
-U 1 1 60FAC21C
-P 7200 5950
-F 0 "MX17" H 7233 6117 50  0000 C CNN
-F 1 "MX_LED" H 7233 6050 20  0000 C CNN
-F 2 "Keebio-Parts:MX-Alps-Choc-2U-StabFlip" H 7250 6050 50  0001 C CNN
-F 3 "" H 7250 6050 50  0001 C CNN
-	1    7200 5950
-	1    0    0    -1
-$EndComp
-$Comp
-L Device:D_Small D20
-U 1 1 60FAC222
-P 7150 6250
-F 0 "D20" V 7196 6180 50  0000 R CNN
-F 1 "D_Small" V 7105 6180 50  0000 R CNN
-F 2 "Diode_SMD:D_SOD-123" V 7150 6250 50  0001 C CNN
-F 3 "~" V 7150 6250 50  0001 C CNN
-	1    7150 6250
-	0    -1   -1   0
-$EndComp
-$Comp
 L kicad-keyboard-parts:MX_LED MX21
 U 1 1 60FAC228
-P 7650 5950
-F 0 "MX21" H 7683 6117 50  0000 C CNN
-F 1 "MX_LED" H 7683 6050 20  0000 C CNN
-F 2 "Keebio-Parts:MX-Alps-Choc-2U-StabFlip" H 7700 6050 50  0001 C CNN
-F 3 "" H 7700 6050 50  0001 C CNN
-	1    7650 5950
+P 8100 5950
+F 0 "MX21" H 8133 6117 50  0000 C CNN
+F 1 "MX_LED" H 8133 6050 20  0000 C CNN
+F 2 "Keebio-Parts:MX-Alps-Choc-2U-StabFlip" H 8150 6050 50  0001 C CNN
+F 3 "" H 8150 6050 50  0001 C CNN
+	1    8100 5950
 	1    0    0    -1
 $EndComp
@@
 L Device:D_Small D24
 U 1 1 60FAC22E
-P 7600 6250
-F 0 "D24" V 7646 6180 50  0000 R CNN
-F 1 "D_Small" V 7555 6180 50  0000 R CNN
-F 2 "Diode_SMD:D_SOD-123" V 7600 6250 50  0001 C CNN
-F 3 "~" V 7600 6250 50  0001 C CNN
-	1    7600 6250
-	0    -1   -1   0
-$EndComp
-$Comp
-L kicad-keyboard-parts:MX_LED MX25
-U 1 1 60FAC234
-P 8100 5950
-F 0 "MX25" H 8133 6117 50  0000 C CNN
-F 1 "MX_LED" H 8133 6050 20  0000 C CNN
-F 2 "Keebio-Parts:MX-Alps-Choc-1U-NoLED" H 8150 6050 50  0001 C CNN
-F 3 "" H 8150 6050 50  0001 C CNN
-	1    8100 5950
-	1    0    0    -1
-$EndComp
-$Comp
-L Device:D_Small D28
-U 1 1 60FAC23A
 P 8050 6250
-F 0 "D28" V 8096 6180 50  0000 R CNN
+F 0 "D24" V 8096 6180 50  0000 R CNN
 F 1 "D_Small" V 8005 6180 50  0000 R CNN
 F 2 "Diode_SMD:D_SOD-123" V 8050 6250 50  0001 C CNN
 F 3 "~" V 8050 6250 50  0001 C CNN
 	1    8050 6250
+	0    -1   -1   0
+$EndComp
+$Comp
+L kicad-keyboard-parts:MX_LED MX25
+U 1 1 60FAC234
+P 8550 5950
+F 0 "MX25" H 8583 6117 50  0000 C CNN
+F 1 "MX_LED" H 8583 6050 20  0000 C CNN
+F 2 "Keebio-Parts:MX-Alps-Choc-1U-NoLED" H 8600 6050 50  0001 C CNN
+F 3 "" H 8600 6050 50  0001 C CNN
+	1    8550 5950
+	1    0    0    -1
+$EndComp
+$Comp
+L Device:D_Small D28
+U 1 1 60FAC23A
+P 8500 6250
+F 0 "D28" V 8546 6180 50  0000 R CNN
+F 1 "D_Small" V 8455 6180 50  0000 R CNN
+F 2 "Diode_SMD:D_SOD-123" V 8500 6250 50  0001 C CNN
+F 3 "~" V 8500 6250 50  0001 C CNN
+	1    8500 6250
 	0    -1   -1   0
 $EndComp
@@
 Text GLabel 9600 3700 1    50   Input ~ 0
 col9
-Text GLabel 10850 2750 1    50   Input ~ 0
-col2
 Wire Wire Line
 	10850 2750 10850 2850
@@
 Wire Wire Line
 	6900 4650 6900 5300
-Connection ~ 6900 5300
-Wire Wire Line
-	6900 5300 6900 5950
 Wire Wire Line
 	7350 3700 7350 3950
@@
 Wire Wire Line
 	7350 4650 7350 5300
-Connection ~ 7350 5300
-Wire Wire Line
-	7350 5300 7350 5950
+Wire Wire Line
+	6900 5300 6900 5950
 Wire Wire Line
 	7800 3700 7800 3950
@@
 Wire Wire Line
 	7800 4650 7800 5300
-Connection ~ 7800 5300
-Wire Wire Line
-	7800 5300 7800 5950
+Wire Wire Line
+	8250 5300 8250 5950
 Wire Wire Line
 	8250 3700 8250 3950
@@
 Wire Wire Line
 	8250 4650 8250 5300
-Connection ~ 8250 5300
-Wire Wire Line
-	8250 5300 8250 5950
 Wire Wire Line
 	8700 3700 8700 3950
@@
 Wire Wire Line
 	8950 5700 9400 5700
-Wire Wire Line
-	5200 6350 6700 6350
-Connection ~ 6700 6350
-Wire Wire Line
-	6700 6350 7150 6350
-Connection ~ 7150 6350
-Wire Wire Line
-	7150 6350 7600 6350
-Connection ~ 7600 6350
-Wire Wire Line
-	7600 6350 8050 6350
 Text GLabel 3450 2000 0    50   Input ~ 0
 sda
@@
 Wire Wire Line
 	7900 2350 8050 2350
-Text GLabel 1800 2200 0    50   Input ~ 0
+Text GLabel 1800 1900 0    50   Input ~ 0
 row0
-Text GLabel 1800 2300 0    50   Input ~ 0
+Text GLabel 1800 1800 0    50   Input ~ 0
 row1
+Text GLabel 1800 1700 0    50   Input ~ 0
+row2
+Text GLabel 1800 1600 0    50   Input ~ 0
+row3
+Text GLabel 3050 1500 2    50   Input ~ 0
+col0
+Text GLabel 3050 1600 2    50   Input ~ 0
+col1
+Text GLabel 3050 1900 2    50   Input ~ 0
+col2
 Text GLabel 3050 2200 2    50   Input ~ 0
-row2
-Text GLabel 3050 1900 2    50   Input ~ 0
-row3
-Text GLabel 1800 2600 0    50   Input ~ 0
-col0
-Text GLabel 1800 2500 0    50   Input ~ 0
-col1
-Text GLabel 1800 2400 0    50   Input ~ 0
-col2
+col3
 Text GLabel 3050 2400 2    50   Input ~ 0
-col3
-Text GLabel 3050 2500 2    50   Input ~ 0
 col4
-Text GLabel 1800 2100 0    50   Input ~ 0
-col5
-Text GLabel 1800 1900 0    50   Input ~ 0
-col6
-Text GLabel 1800 1800 0    50   Input ~ 0
-col7
-Text GLabel 1800 1700 0    50   Input ~ 0
-col8
-Text GLabel 1800 1600 0    50   Input ~ 0
-col9
 Wire Wire Line
 	1050 6350 1050 6400
@@
 Wire Wire Line
 	750  6400 750  6450
+Wire Wire Line
+	3050 2800 3200 2800
+Wire Wire Line
+	1650 2800 1800 2800
+Wire Wire Line
+	1500 2700 1800 2700
+Wire Wire Line
+	1500 1500 1800 1500
+$Comp
+L MINEW_MS88SF2:MS88SF2 U2
+U 1 1 60C5FFDB
+P 2450 2150
+F 0 "U2" H 2425 3067 50  0000 C CNN
+F 1 "MS88SF2" H 2425 2976 50  0000 C CNN
+F 2 "ms88sf2_oreore:MINEW_MS88SF2" H 2450 2200 50  0001 C CNN
+F 3 "" H 2450 2200 50  0001 C CNN
+	1    2450 2150
+	1    0    0    -1
+$EndComp
+$Comp
+L power:GND #PWR0105
+U 1 1 60C8E0D5
+P 1500 1500
+F 0 "#PWR0105" H 1500 1250 50  0001 C CNN
+F 1 "GND" H 1505 1327 50  0000 C CNN
+F 2 "" H 1500 1500 50  0001 C CNN
+F 3 "" H 1500 1500 50  0001 C CNN
+	1    1500 1500
+	1    0    0    -1
+$EndComp
+Wire Wire Line
+	8700 5300 8700 5950
+Connection ~ 8700 5300
+Wire Wire Line
+	6450 5300 6450 5950
+Connection ~ 6450 5300
+Wire Wire Line
+	5200 6350 6250 6350
+Connection ~ 6250 6350
+Wire Wire Line
+	6250 6350 6700 6350
+Connection ~ 8050 6350
+Wire Wire Line
+	8050 6350 8500 6350
+Connection ~ 8250 5300
+Connection ~ 6700 6350
+Connection ~ 6900 5300
+Wire Wire Line
+	6700 6350 8050 6350
+Text GLabel 10850 2750 1    50   Input ~ 0
+col5
+Text GLabel 1800 2300 0    50   Input ~ 0
+col7
+Text GLabel 1800 2200 0    50   Input ~ 0
+col8
+Text GLabel 1800 2100 0    50   Input ~ 0
+col9
+Text GLabel 1800 2400 0    50   Input ~ 0
+col6
+Text GLabel 1800 2500 0    50   Input ~ 0
+col5
+$Comp
+L power:GND #PWR0110
+U 1 1 60CBF5F2
+P 1500 2700
+F 0 "#PWR0110" H 1500 2450 50  0001 C CNN
+F 1 "GND" V 1505 2572 50  0000 R CNN
+F 2 "" H 1500 2700 50  0001 C CNN
+F 3 "" H 1500 2700 50  0001 C CNN
+	1    1500 2700
+	0    1    1    0
+$EndComp
 $EndSCHEMATC
