File: kicad/le_chiff_ble/le_chiff_ble.kicad_pcb (KiCad board)
At the start: 2 copper layers, 228.4 x 85 mm, 117 parts, among them J2 BL_CONN, Q1 AO3401A, SW1 ON_OFF, SW2 SW_RESET, SW3 Rotary_Encoder_Switch, U1 TP4056, U2 MS88SF2, U3 XC6206PxxxMR-Regulator_Linear, U4 DW01A, U5 FS8205, U6 USBLC6-2SC6

Commit message: saved and have to commit
Routing:
- net col2: track 242.6 -> 240.5 mm
- net GND: vias 33 -> 31
Other:
- board text added: "die Zivilisation nur eine sehr dünne Decke ist, die sehr schnell abblättert.“ - Fritz Bauer"
- board text added: "„Ich glaube, es ist eine traurige Wahrheit, dass wir unserem Affenzustand noch sehr nahe sind und dass"
Changed lines of the file:
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@@
   (general
     (thickness 1.6)
-    (drawings 78)
-    (tracks 1212)
+    (drawings 80)
+    (tracks 1216)
     (zones 0)
     (modules 117)
@@
   (module graphics:mangoiv (layer B.Cu)
     (at 151.379425 123.443326 270)
-    (fp_text reference G*** (at 0 0 270) (layer B.SilkS) hide
+    (fp_text reference G*** (at 0 0 270) (layer B.Mask) hide
       (effects (font (size 1.524 1.524) (thickness 0.3)) (justify mirror))
     )
-    (fp_text value LOGO (at 0.75 0 270) (layer B.SilkS) hide
+    (fp_text value LOGO (at 0.75 0 270) (layer B.Mask) hide
       (effects (font (size 1.524 1.524) (thickness 0.3)) (justify mirror))
     )
@@
     )
   )
+  (gr_text "die Zivilisation nur eine sehr dünne Decke ist, \ndie sehr schnell abblättert.“ - Fritz Bauer " (at 134.379425 66.443326 -11) (layer B.Mask)
+    (effects (font (size 1 1) (thickness 0.2)) (justify left mirror))
+  )
+  (gr_text "„Ich glaube, es ist eine traurige Wahrheit, dass wir \nunserem Affenzustand noch sehr nahe sind und dass " (at 154.629425 66.693326 11) (layer B.Mask)
+    (effects (font (size 1 1) (thickness 0.2)) (justify right mirror))
+  )
   (gr_text RESET (at 147.474663 91.943326) (layer B.SilkS)
     (effects (font (size 1 1) (thickness 0.25)) (justify left mirror))
@@
   (segment (start 157.739425 118.553326) (end 158.379425 119.193326) (width 0.381) (layer F.Cu) (net 3))
   (segment (start 158.379425 119.193326) (end 160.379425 119.193326) (width 0.381) (layer F.Cu) (net 3))
-  (via (at 132.879425 67.943326) (size 0.8) (drill 0.4) (layers F.Cu B.Cu) (net 3))
   (via (at 94.879425 58.693326) (size 0.8) (drill 0.4) (layers F.Cu B.Cu) (net 3))
   (via (at 128.629425 107.193326) (size 0.8) (drill 0.4) (layers F.Cu B.Cu) (net 3))
@@
   (via (at 137.879425 74.943326) (size 0.8) (drill 0.4) (layers F.Cu B.Cu) (net 3))
   (via (at 119.579425 136.873666) (size 0.8) (drill 0.4) (layers F.Cu B.Cu) (net 3))
-  (via (at 113.379425 67.693326) (size 0.8) (drill 0.4) (layers F.Cu B.Cu) (net 3))
-  (via (at 94.629425 66.193326) (size 0.8) (drill 0.4) (layers F.Cu B.Cu) (net 3))
   (via (at 130.129425 74.443326) (size 0.8) (drill 0.4) (layers F.Cu B.Cu) (net 3))
+  (via (at 112.129425 75.693326) (size 0.8) (drill 0.4) (layers F.Cu B.Cu) (net 3))
   (segment (start 142.879425 66.693326) (end 141.879425 67.693326) (width 0.381) (layer F.Cu) (net 4))
   (segment (start 145.690425 66.693326) (end 142.879425 66.693326) (width 0.381) (layer F.Cu) (net 4))
@@
   (segment (start 230.379425 73.593326) (end 237.379425 80.593326) (width 0.25) (layer B.Cu) (net 14))
   (segment (start 217.379425 73.593326) (end 230.379425 73.593326) (width 0.25) (layer B.Cu) (net 14))
-  (segment (start 126.379425 82.843326) (end 110.129425 82.843326) (width 0.25) (layer B.Cu) (net 14))
-  (segment (start 128.879425 85.343326) (end 126.379425 82.843326) (width 0.25) (layer B.Cu) (net 14))
-  (segment (start 102.279425 75.843326) (end 91.879425 75.843326) (width 0.25) (layer B.Cu) (net 14))
-  (segment (start 109.279425 82.843326) (end 102.279425 75.843326) (width 0.25) (layer B.Cu) (net 14))
-  (segment (start 110.129425 82.843326) (end 109.279425 82.843326) (width 0.25) (layer B.Cu) (net 14))
   (segment (start 75.379219 75.343532) (end 72.379425 78.343326) (width 0.25) (layer B.Cu) (net 14))
   (segment (start 91.379631 75.343532) (end 75.379219 75.343532) (width 0.25) (layer B.Cu) (net 14))
@@
   (via (at 162.979425 85.343326) (size 0.8) (drill 0.4) (layers F.Cu B.Cu) (net 14))
   (segment (start 161.379425 85.343326) (end 162.979425 85.343326) (width 0.25) (layer B.Cu) (net 14))
-  (segment (start 159.354426 83.318327) (end 161.379425 85.343326) (width 0.25) (layer B.Cu) (net 14))
-  (segment (start 130.904424 83.318327) (end 159.354426 83.318327) (width 0.25) (layer B.Cu) (net 14))
-  (segment (start 128.879425 85.343326) (end 130.904424 83.318327) (width 0.25) (layer B.Cu) (net 14))
   (segment (start 157.019425 124.053326) (end 160.204413 120.868338) (width 0.25) (layer F.Cu) (net 14))
   (segment (start 153.629425 124.053326) (end 157.019425 124.053326) (width 0.25) (layer F.Cu) (net 14))
@@
   (segment (start 167.479425 85.343326) (end 169.979425 82.843326) (width 0.25) (layer B.Cu) (net 14))
   (segment (start 162.979425 85.343326) (end 167.479425 85.343326) (width 0.25) (layer B.Cu) (net 14))
+  (segment (start 121.779425 82.843326) (end 110.129425 82.843326) (width 0.25) (layer B.Cu) (net 14))
+  (segment (start 124.279425 85.343326) (end 121.779425 82.843326) (width 0.25) (layer B.Cu) (net 14))
+  (segment (start 128.879425 85.343326) (end 124.279425 85.343326) (width 0.25) (layer B.Cu) (net 14))
+  (segment (start 99.529425 75.843326) (end 91.879425 75.843326) (width 0.25) (layer B.Cu) (net 14))
+  (segment (start 106.529425 82.843326) (end 99.529425 75.843326) (width 0.25) (layer B.Cu) (net 14))
+  (segment (start 110.129425 82.843326) (end 106.529425 82.843326) (width 0.25) (layer B.Cu) (net 14))
+  (segment (start 128.879425 85.343326) (end 130.115835 85.343326) (width 0.25) (layer B.Cu) (net 14))
+  (segment (start 130.115835 85.343326) (end 132.140834 83.318327) (width 0.25) (layer B.Cu) (net 14))
+  (segment (start 132.140834 83.318327) (end 159.354426 83.318327) (width 0.25) (layer B.Cu) (net 14))
+  (segment (start 159.354426 83.318327) (end 161.379425 85.343326) (width 0.25) (layer B.Cu) (net 14))
   (segment (start 41.416788 83.055514) (end 40.285035 83.055514) (width 0.25) (layer B.Cu) (net 15))
   (segment (start 42.997952 81.47435) (end 41.416788 83.055514) (width 0.25) (layer B.Cu) (net 15))
@@
   (segment (start 118.661044 69.998903) (end 117.340595 69.998903) (width 0.25) (layer B.Cu) (net 30))
   (segment (start 121.531677 67.12827) (end 118.661044 69.998903) (width 0.25) (layer B.Cu) (net 30))
-  (segment (start 126.439708 82.043326) (end 128.879425 82.043326) (width 0.25) (layer B.Cu) (net 30))
-  (segment (start 117.340595 72.944213) (end 126.439708 82.043326) (width 0.25) (layer B.Cu) (net 30))
-  (segment (start 117.340595 69.998903) (end 117.340595 72.944213) (width 0.25) (layer B.Cu) (net 30))
+  (segment (start 128.829414 81.993315) (end 128.879425 82.043326) (width 0.25) (layer B.Cu) (net 30))
+  (segment (start 117.420526 73.024144) (end 126.389697 81.993315) (width 0.25) (layer B.Cu) (net 30))
+  (segment (start 117.420526 70.078834) (end 117.420526 73.024144) (width 0.25) (layer B.Cu) (net 30))
+  (segment (start 126.389697 81.993315) (end 128.829414 81.993315) (width 0.25) (layer B.Cu) (net 30))
+  (segment (start 117.340595 69.998903) (end 117.420526 70.078834) (width 0.25) (layer B.Cu) (net 30))
   (segment (start 117.628903 87.617436) (end 116.49715 87.617436) (width 0.25) (layer B.Cu) (net 31))
   (segment (start 119.210067 86.036272) (end 117.628903 87.617436) (width 0.25) (layer B.Cu) (net 31))
@@
   (segment (start 145.625427 74.393326) (end 139.825427 80.193326) (width 0.25) (layer F.Cu) (net 57))
   (segment (start 150.129425 74.393326) (end 145.625427 74.393326) (width 0.25) (layer F.Cu) (net 57))
-  (segment (start 107.879425 63.193326) (end 91.741677 63.193326) (width 0.25) (layer B.Cu) (net 57))
-  (segment (start 110.379425 65.693326) (end 107.879425 63.193326) (width 0.25) (layer B.Cu) (net 57))
-  (segment (start 126.129425 65.693326) (end 110.379425 65.693326) (width 0.25) (layer B.Cu) (net 57))
-  (segment (start 134.129425 73.693326) (end 126.129425 65.693326) (width 0.25) (layer B.Cu) (net 57))
+  (segment (start 110.379425 68.193326) (end 105.379425 63.193326) (width 0.25) (layer B.Cu) (net 57))
+  (segment (start 130.379425 84.443326) (end 124.379425 84.443326) (width 0.25) (layer B.Cu) (net 57))
+  (segment (start 132.379425 82.443326) (end 130.379425 84.443326) (width 0.25) (layer B.Cu) (net 57))
+  (segment (start 110.379425 70.443326) (end 110.379425 68.193326) (width 0.25) (layer B.Cu) (net 57))
+  (segment (start 124.379425 84.443326) (end 110.379425 70.443326) (width 0.25) (layer B.Cu) (net 57))
+  (segment (start 134.129425 82.443326) (end 132.379425 82.443326) (width 0.25) (layer B.Cu) (net 57))
   (segment (start 91.741677 63.193326) (end 89.002572 60.454221) (width 0.25) (layer B.Cu) (net 57))
-  (segment (start 134.129425 82.443326) (end 134.129425 73.693326) (width 0.25) (layer B.Cu) (net 57))
+  (segment (start 105.379425 63.193326) (end 91.741677 63.193326) (width 0.25) (layer B.Cu) (net 57))
   (segment (start 135.039425 121.853326) (end 131.063393 117.877294) (width 0.25) (layer F.Cu) (net 58))
   (via (at 131.063393 117.877294) (size 0.8) (drill 0.4) (layers F.Cu B.Cu) (net 58))

Commit message: started rerouting
Parts:
- removed G***: LOGO, graphics:tomina
- removed G***: LOGO, graphics:mangoiv
- removed G***: LOGO, graphics:logo_big
- D10, D11, D12, D13, D14, D15, D16, D17, D18, D19, D20, D21, D22, D23, D24, D25, D26, D27, D28, D29, D30, D31, D32, D33, D34, D35, D36, D37, D38, D4, D5, D6, D7, D8, D9: moved to F.Cu
- moved R3 4.50 mm to (160.1, 124.7)
- moved R2 4.50 mm to (160.1, 122.2)
- moved D23 1.25 mm to (166.6, 120.7)
- moved D22 1.03 mm to (164.6, 102.2)
- moved D24 0.46 mm to (173.0, 129.0)
- moved D38 0.38 mm to (135.8, 83.4)
- moved C2 0.05 mm to (160.1, 117.7)
Connections:
- MX13 pad 1: col3 -> col2
- MX17 pad 1: col4 -> col3
- MX21 pad 1: col5 -> col6
- MX25 pad 1: col6 -> col7
- MX28 pad 2: Net-(D31-Pad2) -> Net-(MX28-Pad2)
- MX35 pad 1: col2 -> col5
- SW3 pad S1: col2 -> col5
- U2 pad 10: col2 -> col6
- U2 pad 11: col1 -> col5
- U2 pad 12: col0 -> encA
- U2 pad 18: col4 -> encB
- U2 pad 19: col3 -> col4
- U2 pad 2: col9 -> row3
- U2 pad 21: row2 -> col3
- U2 pad 24: row3 -> col2
- U2 pad 27: encB -> col1
- U2 pad 28: encA -> col0
- U2 pad 3: col8 -> row2
- U2 pad 4: col7 -> row1
- U2 pad 5: col6 -> row0
- U2 pad 7: col5 -> col9
- U2 pad 8: row0 -> col8
- U2 pad 9: row1 -> col7
Routing:
- net vbus: track 225.1 -> 78.3 mm, vias 6 -> 2
- net col2: track 240.5 -> 127.0 mm, vias 3 -> 1
- net Net-(D1-Pad1): track 112.7 -> 0.04 mm, vias 4 -> 0
- net GND: track 259.9 -> 164.1 mm, vias 31 -> 1
- net row1: track 264.0 -> 174.0 mm, vias 1 -> 2
- net Net-(D2-Pad1): track 90.0 -> 0.00 mm, vias 3 -> 0
- net row2: track 231.6 -> 142.2 mm, vias 1 -> 2
- net +3V3: track 101.2 -> 14.0 mm, vias 4 -> 1
- net encB: track 65.0 -> 0.00 mm, vias 2 -> 0
- net col6: track 158.3 -> 96.4 mm, vias 3 -> 1
- net encA: track 59.3 -> 0.00 mm, vias 2 -> 0
- net row3: track 182.0 -> 133.7 mm, vias 4 -> 2
- net col7: track 165.2 -> 125.7 mm, vias 0 -> 1
- net col3: track 127.8 -> 98.7 mm, vias 4 -> 1
- net col4: track 101.4 -> 74.8 mm, vias 2 -> 1
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- removed copper zone on B.Cu, net GND
- removed copper zone on F.Cu, net GND
